File: KiCad/RX_SKETCHES/ESP_32_IEM_RIG_RX_VER_1.0.kicad_pcb (KiCad board)
At the start: 2 copper layers, 55.2 x 90.5 mm, 69 parts, among them J1 AudioJack3, J6 USB_C_Receptacle_USB2.0_16P, Q1 S8050, Q2 S8050, SW2 FILTER_MODE, SW3 SOFT_MUTE, SW4 ON/OFF, U1 PCM5102, U2 ESP32-WROOM-32U, U3 MAX97220AETE_T, U4 LM3940IMPX-3.3_NOPB, U5 CP2102C-Axx-xQFN24

Commit message: FINISHED_RX_V1_Schematics!
Finished V1 of RX PCBs!
Other:
- board text added: "Designed by Damian Muschamp. https://github.com/dlmuschamp/ESP32IEMPack.git"
- board text removed: "https://github.com/dlmuschamp/ESP32IEMPack.git"
