File: KiCad/RX_SKETCHES/amp.kicad_sch (KiCad schematic)
At the start: 19 parts, among them J1 AudioJack3, U3 MAX97220AETE_T

Commit message: Rewire RX hierarchical labels and mark proto DNP parts.
Keep the rotated WROOM-32U and breadboard I2S GPIOs, but attach
ESP_EN/IO0, UART, and BCK/DIN/LRCLK to the pins that actually sit
there after the 270° rotate. Move PCM5102 I2S off FMT/DEMP/XSMT,
put amp shutdown on ~{SHDN}, keep the datasheet 470R+2.2nF filter,
DNP the experimental pot pad and MAX97220A input resistors, and
switch schematic passives to 0805 for hand assembly.

Co-authored-by: luciano <dlmuschamp@users.noreply.github.com>
Parts:
- C1, C10, C2, C3, C4, C6, C7, C8, C9: footprint Capacitor_SMD:C_0201_0603Metric -> Capacitor_SMD:C_0805_2012Metric
- R1, R10, R2, R3, R4, R5, R6, R9: footprint Resistor_SMD:R_0201_0603Metric -> Resistor_SMD:R_0805_2012Metric; now not fitted
Connections:
- net SHDN_SIGNAL: now also U3.4 (C1N); no longer U3.16 (~{SHDN})
- net at U3.2 (C1P): no longer C7.1
- net at C7.2: now also U3.16 (~{SHDN}); no longer U3.4 (C1N)
Other:
- note added: "SHDN_SIGNAL -> pin 16 ~{SHDN} (active low). C7 1uF is the C1P-C1N flying cap, not on SHDN. R1-R6, R9, R10 are DNP on hand-built protos so gain / input attenuation can be socketed. Populate them (start 10k) on a fully assembled board. MAX97220A gain is fixed +3.5 dB; these Rs are the single-ended input network, not an IC gain pin. Use MAX97220D if you want resistor-programmed gain. Zin of the A ve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"
- moved on the sheet: C7
Changed lines of the file:
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@@
 	(wire
 		(pts
-			(xy 88.9 67.31) (xy 88.9 69.85)
+			(xy 88.9 59.69) (xy 88.9 62.23)
 		)
 		(stroke
@@
 	(wire
 		(pts
-			(xy 96.52 67.31) (xy 88.9 67.31)
+			(xy 96.52 62.23) (xy 88.9 62.23)
 		)
 		(stroke
@@
 			(width 0)
 			(type default)
+		)
+	)
+	(text "SHDN_SIGNAL -> pin 16 ~{SHDN} (active low).\nC7 1uF is the C1P-C1N flying cap, not on SHDN.\n\nR1-R6, R9, R10 are DNP on hand-built protos\nso gain / input attenuation can be socketed.\nPopulate them (start 10k) on a fully assembled board.\nMAX97220A gain is fixed +3.5 dB; these Rs are the\nsingle-ended input network, not an IC gain pin.\nUse MAX97220D if you want resistor-programmed gain.\n\nZin of the A version is ~10 kOhm, which matches\nthe PCM5102 470R + 2.2nF output filter."
+		(exclude_from_sim no)
+		(at 20.32 20.32 0)
+		(effects
+			(font
+				(size 1.27 1.27)
+			)
+			(justify left)
 		)
 	)
@@
 	(hierarchical_label "SHDN_SIGNAL"
 		(shape input)
-		(at 96.52 62.23 180)
+		(at 96.52 67.31 180)
 		(effects
 			(font
@@
 			)
 		)
-		(property "Footprint" "Capacitor_SMD:C_0201_0603Metric"
+		(property "Footprint" "Capacitor_SMD:C_0805_2012Metric"
 			(at 50.8 58.7248 0)
 			(hide yes)
@@
 			)
 		)
-		(property "Footprint" "Capacitor_SMD:C_0201_0603Metric"
+		(property "Footprint" "Capacitor_SMD:C_0805_2012Metric"
 			(at 120.65 20.6248 0)
 			(hide yes)
@@
 		(on_board yes)
 		(in_pos_files yes)
-		(dnp no)
+		(dnp yes)
 		(fields_autoplaced yes)
 		(property "Reference" "R5"
@@
 			)
 		)
-		(property "Footprint" "Resistor_SMD:R_0201_0603Metric"
+		(property "Footprint" "Resistor_SMD:R_0805_2012Metric"
 			(at 61.214 58.674 90)
 			(hide yes)
@@
 		(on_board yes)
 		(in_pos_files yes)
-		(dnp no)
+		(dnp yes)
 		(fields_autoplaced yes)
 		(property "Reference" "R3"
@@
 			)
 		)
-		(property "Footprint" "Resistor_SMD:R_0201_0603Metric"
+		(property "Footprint" "Resistor_SMD:R_0805_2012Metric"
 			(at 69.596 66.294 90)
 			(hide yes)
@@
 		(on_board yes)
 		(in_pos_files yes)
-		(dnp no)
+		(dnp yes)
 		(fields_autoplaced yes)
 		(property "Reference" "R4"
@@
 			)
 		)
-		(property "Footprint" "Resistor_SMD:R_0201_0603Metric"
+		(property "Footprint" "Resistor_SMD:R_0805_2012Metric"
 			(at 61.214 45.974 90)
 			(hide yes)
@@
 		(on_board yes)
 		(in_pos_files yes)
-		(dnp no)
+		(dnp yes)
 		(fields_autoplaced yes)
 		(property "Reference" "R2"
@@
 			)
 		)
-		(property "Footprint" "Resistor_SMD:R_0201_0603Metric"
+		(property "Footprint" "Resistor_SMD:R_0805_2012Metric"
 			(at 61.214 98.044 90)
 			(hide yes)
@@
 			)
 		)
-		(property "Footprint" "Capacitor_SMD:C_0201_0603Metric"
+		(property "Footprint" "Capacitor_SMD:C_0805_2012Metric"
 			(at 151.13 79.0448 0)
 			(hide yes)
@@
 			)
 		)
-		(property "Footprint" "Capacitor_SMD:C_0201_0603Metric"
+		(property "Footprint" "Capacitor_SMD:C_0805_2012Metric"
 			(at 151.13 20.6248 0)
 			(hide yes)
@@
 			)
 		)
-		(property "Footprint" "Capacitor_SMD:C_0201_0603Metric"
+		(property "Footprint" "Capacitor_SMD:C_0805_2012Metric"
 			(at 50.8 46.0248 0)
 			(hide yes)
@@
 			)
 		)
-		(property "Footprint" "Capacitor_SMD:C_0201_0603Metric"
+		(property "Footprint" "Capacitor_SMD:C_0805_2012Metric"
 			(at 50.8 85.3948 0)
 			(hide yes)
@@
 		(on_board yes)
 		(in_pos_files yes)
-		(dnp no)
+		(dnp yes)
 		(fields_autoplaced yes)
 		(property "Reference" "R1"
@@
 			)
 		)
-		(property "Footprint" "Resistor_SMD:R_0201_0603Metric"
+		(property "Footprint" "Resistor_SMD:R_0805_2012Metric"
 			(at 101.854 32.004 90)
 			(hide yes)
@@
 			)
 		)
-		(property "Footprint" "Capacitor_SMD:C_0201_0603Metric"
+		(property "Footprint" "Capacitor_SMD:C_0805_2012Metric"
 			(at 50.8 98.0948 0)
 			(hide yes)
@@
 	(symbol
 		(lib_id "Device:C")
-		(at 92.71 69.85 270)
+		(at 92.71 59.69 270)
 		(unit 1)
 		(body_style 1)
@@
 		(dnp no)
 		(property "Reference" "C7"
-			(at 92.71 74.422 90)
+			(at 92.71 64.262 90)
 			(show_name no)
 			(do_not_autoplace no)
@@
 		)
 		(property "Value" "1u"
-			(at 92.71 76.708 90)
-			(show_name no)
-			(do_not_autoplace no)
-			(effects
-				(font
-					(size 1.27 1.27)
-				)
-			)
-		)
-		(property "Footprint" "Capacitor_SMD:C_0201_0603Metric"
+			(at 92.71 66.548 90)
+			(show_name no)
+			(do_not_autoplace no)
+			(effects
+				(font
+					(size 1.27 1.27)
+				)
+			)
+		)
+		(property "Footprint" "Capacitor_SMD:C_0805_2012Metric"
 			(at 88.9 70.8152 0)
 			(hide yes)
@@
 			)
 		)
-		(property "Footprint" "Capacitor_SMD:C_0201_0603Metric"
+		(property "Footprint" "Capacitor_SMD:C_0805_2012Metric"
 			(at 151.13 66.3448 0)
 			(hide yes)
@@
 		(on_board yes)
 		(in_pos_files yes)
-		(dnp no)
+		(dnp yes)
 		(fields_autoplaced yes)
 		(property "Reference" "R6"
@@
 			)
 		)
-		(property "Footprint" "Resistor_SMD:R_0201_0603Metric"
+		(property "Footprint" "Resistor_SMD:R_0805_2012Metric"
 			(at 61.214 85.344 90)
 			(hide yes)
@@
 		(on_board yes)
 		(in_pos_files yes)
-		(dnp no)
+		(dnp yes)
 		(fields_autoplaced yes)
 		(property "Reference" "R9"
@@
 			)
 		)
-		(property "Footprint" "Resistor_SMD:R_0201_0603Metric"
+		(property "Footprint" "Resistor_SMD:R_0805_2012Metric"
 			(at 69.596 78.994 90)
 			(hide yes)
@@
 		(on_board yes)
 		(in_pos_files yes)
-		(dnp no)
+		(dnp yes)
 		(fields_autoplaced yes)
 		(property "Reference" "R10"
@@
 			)
 		)
-		(property "Footprint" "Resistor_SMD:R_0201_0603Metric"
+		(property "Footprint" "Resistor_SMD:R_0805_2012Metric"
 			(at 106.934 100.584 90)
 			(hide yes)

Commit message: Align RX passives and analog nets with the part datasheets.
Put every R/C on the 0805 HandSolder footprint. Rewire the PCM5102
470R filter onto OUTL/OUTR, decouple LDOO, and land the flying cap
on CAPP/CAPM. Move the headphone jack off PVSS/SVSS onto OUTL/OUTR
with a PVSS hold cap. Tie CP2102C VIO to VDD, pull RST up, add the
LM3940 0.47uF Cin, and pull IO0 up for normal boot.

Co-authored-by: luciano <dlmuschamp@users.noreply.github.com>
Parts:
- added C29: 1u, Capacitor_SMD:C_0805_2012Metric_Pad1.15x1.40mm_HandSolder, symbol Device:C
- C1, C10, C2, C3, C4, C6, C7, C8, C9: footprint Capacitor_SMD:C_0805_2012Metric -> Capacitor_SMD:C_0805_2012Metric_Pad1.15x1.40mm_HandSolder
- R1, R10, R2, R3, R4, R5, R6, R9: footprint Resistor_SMD:R_0805_2012Metric -> Resistor_SMD:R_0805_2012Metric_Pad1.20x1.40mm_HandSolder
Connections:
- net GND: now also C10.1, C6.1, J1.R, J1.T, U3.11 (SVSS), U3.5 (PVSS), C29.2
- removed net AMP_OUT_L: J1.T, R1.2, U3.12 (OUTL)
- net AMP_OUT_R: no longer names the net of R10.2, U3.10 (OUTR)
- net AMP_OUT_R: now also U3.12 (OUTL), C29.1; no longer J1.R
Other:
- note added: "SHDN_SIGNAL -> pin 16 ~{SHDN} (active low). C7 1uF is the C1P-C1N flying cap, not on SHDN. R1-R6, R9, R10 are DNP on hand-built protos so gain / input attenuation can be socketed. Populate them (start 10k) on a fully assembled board. MAX97220A gain is fixed +3.5 dB; these Rs are the single-ended input network, not an IC gain pin. Use MAX97220D if you want resistor-programmed gain. Jack: Tip=OUTL,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"
- note removed: "SHDN_SIGNAL -> pin 16 ~{SHDN} (active low). C7 1uF is the C1P-C1N flying cap, not on SHDN. R1-R6, R9, R10 are DNP on hand-built protos so gain / input attenuation can be socketed. Populate them (start 10k) on a fully assembled board. MAX97220A gain is fixed +3.5 dB; these Rs are the single-ended input network, not an IC gain pin. Use MAX97220D if you want resistor-programmed gain. Zin of the A ve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"
