File: KiCad/RX_SKETCHES/amp.kicad_sch (KiCad schematic)
At the start: 20 parts, among them J1 AudioJack3, U3 MAX97220AETE_T

Commit message: WIP: RX schematic review — restore DAC/amp, fix ESP nets, log revisions.
Restore dac/amp from main after rotate damage, rename I2S net to DOUT,
mark amp gain Rs DNP, and record change/rationale in docs/hardware_revisions.org.

Co-authored-by: Cursor <cursoragent@cursor.com>
Parts:
- removed C29: 1u, Capacitor_SMD:C_0805_2012Metric_Pad1.15x1.40mm_HandSolder, symbol Device:C
- C1, C10, C2, C3, C4, C6, C7, C8, C9: footprint Capacitor_SMD:C_0805_2012Metric_Pad1.15x1.40mm_HandSolder -> Capacitor_SMD:C_0201_0603Metric
- R1, R10, R2, R3, R4, R5, R6, R9: footprint Resistor_SMD:R_0805_2012Metric_Pad1.20x1.40mm_HandSolder -> Resistor_SMD:R_0201_0603Metric
Connections:
- net GND: no longer C10.1, C6.1, J1.R, J1.T, U3.11 (SVSS), U3.5 (PVSS)
- net SHDN_SIGNAL: now also U3.16 (~{SHDN}); no longer U3.4 (C1N)
- net AMP_OUT_R: now reaches R10.2, U3.10 (OUTR)
- net AMP_OUT_R: now also J1.R; no longer U3.12 (OUTL)
- net at C7.2: now also U3.4 (C1N); no longer U3.16 (~{SHDN})
- net at U3.2 (C1P): now also C7.1
- net AMP_OUT_L: now reaches R1.2
- net AMP_OUT_L: now also J1.T, U3.12 (OUTL)
- new net: C6.1, U3.5 (PVSS)
- new net: C10.1, U3.11 (SVSS)
Other:
- note added: "SHDN_SIGNAL LOW acts as setting the volume to a "true 0%" by shutting off the IEM amp. This is in contrast to the DAC Soft mute which acts as a mute toggle without changing the volume. Amp follows the pseudo-differential input configuration because the DAC output is a single-ended input. R1-R6, R9, R10 are DNP (Do Not Populate) on hand-built protos so gain / input attenuation can be chosen later.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"
- note removed: "SHDN_SIGNAL -> pin 16 ~{SHDN} (active low). C7 1uF is the C1P-C1N flying cap, not on SHDN. R1-R6, R9, R10 are DNP on hand-built protos so gain / input attenuation can be socketed. Populate them (start 10k) on a fully assembled board. MAX97220A gain is fixed +3.5 dB; these Rs are the single-ended input network, not an IC gain pin. Use MAX97220D if you want resistor-programmed gain. Jack: Tip=OUTL,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"
- note removed: "SHDN_SIGNAL LOW acts as setting the volume to a "true 0%" by shutting off the IEM amp. This is in contrast to the DAC Soft mute which acts as a mute toggle without changing the volume. Amp follows the pseudo-differential input configuration because the DAC output is a single-ended input."
- moved on the sheet: C7

Commit message: RX: finish layout, retune gain/coupling, move ESD clamp to unswitched VBUS
Board now passes DRC with zero unconnected items and zero schematic-parity
issues. Remaining 16 violations are footprint-inherent (ESP32 module thermal
via array at 0.2 mm drill, USB-C NPTH-to-pad spacing) and are documented
rather than routed around.

Analog changes, with the reasoning captured in README.org and
docs/hardware_revisions.org so the numbers can be re-checked:

- Gain network populated at RF 4.7k / RIN 47k (-20 dB) instead of DNP 10k.
  Tames the DAC's 2.1 Vrms into sensitive IEMs, unloads the pot taper, and
  moves the coupling corner out of the audible band.
- Coupling caps C1-C4 0.47uF -> 1uF. Corner 7.2 Hz -> 3.4 Hz, and it halves
  the signal developed across the ceramic at 20 Hz, cutting Class-II
  dielectric distortion where it actually occurs.
- D1's third TVS channel moved off the switched +5V rail onto VBUS_RAW. The
  clamp has to sit on the connector pin that is exposed to a finger; behind
  the power switch it went open exactly when the board is most handled.
- SW3 soft mute: XSMT_SEL moved to the throw that puts mute on the south
  slide position. All three switches now follow one rule -- the open throw
  is the safe default (off / quality filter / muted).
- PCM5102 mode pins no longer float: FLT and XSMT get 100k pulldowns, DEMP
  and FMT strap to GND.
- C28 and the four mounting holes added to the schematic to clear parity
  errors against parts that only existed on the PCB.

Also adds a .gitignore so the 24 MB editor .history/ directory and ESP-IDF
build output stop showing up as untracked.

Co-authored-by: Cursor <cursoragent@cursor.com>
Parts:
- added C28: 1u, Capacitor_SMD:C_0805_2012Metric_Pad1.18x1.45mm_HandSolder, symbol Device:C
- C1, C2, C3, C4: value 0.47u -> 1u; footprint Capacitor_SMD:C_0201_0603Metric -> Capacitor_SMD:C_0805_2012Metric_Pad1.18x1.45mm_HandSolder
- C10, C6, C7, C8, C9: footprint Capacitor_SMD:C_0201_0603Metric -> Capacitor_SMD:C_0805_2012Metric_Pad1.18x1.45mm_HandSolder
- R1, R10, R3, R9: value 10k -> 4.7k; footprint Resistor_SMD:R_0201_0603Metric -> Resistor_SMD:R_0805_2012Metric_Pad1.20x1.40mm_HandSolder; now fitted
- R2, R4, R5, R6: value 10k -> 47k; footprint Resistor_SMD:R_0201_0603Metric -> Resistor_SMD:R_0805_2012Metric_Pad1.20x1.40mm_HandSolder; now fitted
Connections:
- net +3V3: now also C28.1
- net GND: now also C28.2
- net AMP_OUT_L: no longer names the net of J1.T, R1.2, U3.12 (OUTL)
- net AMP_OUT_R: no longer names the net of J1.R, R10.2, U3.10 (OUTR)
Other:
- note added: "Left Output"
- note added: "R_F"
- note added: "R_in"
- note added: "Right Output"
- note added: "SHDN_SIGNAL LOW acts as setting the volume to a "true 0%" by shutting off the IEM amp. This is in contrast to the DAC Soft mute which acts as a mute toggle without changing the volume. Amp follows the pseudo-differential input configuration because the DAC output is a single-ended input. R_F (R1,R3,R9,R10) and R_IN (R2,R4,R5,R6) set the gain. Each group must stay matched or the pseudo-differentia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"
- note added: "VOLUME / GAIN BUDGET (full derivation in README.org) R_F = R1,R3,R9,R10 = 4.7k R_IN = R2,R4,R5,R6 = 47k VR1 divider 10k/(470+10k) = -0.40 dB Amp gain 4.7k / 47k = -20.00 dB TOTAL = -20.40 dB (x0.0955) PCM5102A full scale is 2.1 Vrms, so at max volume Vout = 2.1 x 0.0955 = 0.201 Vrms at J1 Peak SPL = IEM dB/Vrms + 20*log10(Vout), and to convert a dB/mW spec: dB/Vrms = dB/mW + 10*log10(1000/Z) KZ Z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"
- note removed: "SHDN_SIGNAL LOW acts as setting the volume to a "true 0%" by shutting off the IEM amp. This is in contrast to the DAC Soft mute which acts as a mute toggle without changing the volume. Amp follows the pseudo-differential input configuration because the DAC output is a single-ended input. R1-R6, R9, R10 are DNP (Do Not Populate) on hand-built protos so gain / input attenuation can be chosen later.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"
