File: KiCad/RX_SKETCHES/amp.kicad_sch (KiCad schematic)
At the start: 19 parts, among them J1 AudioJack3, U3 MAX97220AETE_T

Commit message: RX v1: complete PCB layout, retune analog chain, fix ESD clamp placement
Brings the RX schematic and board up to a fabricable state. DRC is clean:
zero unconnected items, zero schematic-parity issues. The 16 remaining
violations are footprint-inherent and documented rather than worked around
(ESP32-WROOM thermal via array drilled 0.2 mm against a 0.3 mm rule, and
USB-C NPTH-to-pad spacing from the vendor land pattern).

Analog:
- Gain network populated at RF 4.7k / RIN 47k (-20 dB) rather than DNP 10k.
  Tames the PCM5102's 2.1 Vrms into sensitive IEMs, gives the 10k pot a
  4.7x loading ratio instead of 1:1, and lifts the coupling corner clear of
  the audible band.
- Coupling caps C1-C4 raised 0.47uF -> 1uF. Corner 7.2 Hz -> 3.4 Hz, and it
  halves the signal developed across the ceramic at 20 Hz, which is where
  Class-II dielectric distortion actually shows up.
- PCM5102 mode pins no longer float: 100k pulldowns on FLT and XSMT, with
  DEMP and FMT strapped to GND.

Power and protection:
- D1's third TVS channel moved off the switched +5V rail onto VBUS_RAW. An
  ESD clamp has to sit on the connector pin exposed to a finger; behind the
  power switch it disconnected exactly when the board is most likely to be
  handled. The off state is unaffected -- a TVS is open below its standoff
  voltage and SW4 still breaks the rail.
- All three slide switches now follow one rule: the open throw is the safe
  default (powered off / normal-latency filter / muted).

Housekeeping:
- C28 and mounting holes REF1-REF4 added to the schematic, clearing parity
  errors against parts that previously existed only on the PCB.
- Gain, loudness, and filter math written up in README.org with sources so
  the numbers can be re-derived; rationale logged in hardware_revisions.org.
- .gitignore now covers the editor .history/ directory and ESP-IDF build
  output, which were showing up as untracked noise.

Firmware and build artifacts are deliberately excluded from this commit.

Co-authored-b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
Parts:
- added C28: 1u, Capacitor_SMD:C_0805_2012Metric_Pad1.18x1.45mm_HandSolder, symbol Device:C
- C1, C2, C3, C4: value 0.47u -> 1u; footprint Capacitor_SMD:C_0201_0603Metric -> Capacitor_SMD:C_0805_2012Metric_Pad1.18x1.45mm_HandSolder
- C10, C6, C7, C8, C9: footprint Capacitor_SMD:C_0201_0603Metric -> Capacitor_SMD:C_0805_2012Metric_Pad1.18x1.45mm_HandSolder
- R1, R10, R3, R9: value 10k -> 4.7k; footprint Resistor_SMD:R_0201_0603Metric -> Resistor_SMD:R_0805_2012Metric_Pad1.20x1.40mm_HandSolder
- R2, R4, R5, R6: value 10k -> 47k; footprint Resistor_SMD:R_0201_0603Metric -> Resistor_SMD:R_0805_2012Metric_Pad1.20x1.40mm_HandSolder
Connections:
- net +3V3: now also C28.1
- net GND: now also C28.2
- net AMP_OUT_L: no longer names the net of J1.T, R1.2, U3.12 (OUTL)
- net AMP_OUT_R: no longer names the net of J1.R, R10.2, U3.10 (OUTR)
Other:
- note added: "Left Output"
- note added: "R_F"
- note added: "R_in"
- note added: "Right Output"
- note added: "SHDN_SIGNAL LOW acts as setting the volume to a "true 0%" by shutting off the IEM amp. This is in contrast to the DAC Soft mute which acts as a mute toggle without changing the volume. Amp follows the pseudo-differential input configuration because the DAC output is a single-ended input. R_F (R1,R3,R9,R10) and R_IN (R2,R4,R5,R6) set the gain. Each group must stay matched or the pseudo-differentia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"
- note added: "VOLUME / GAIN BUDGET (full derivation in README.org) R_F = R1,R3,R9,R10 = 4.7k R_IN = R2,R4,R5,R6 = 47k VR1 divider 10k/(470+10k) = -0.40 dB Amp gain 4.7k / 47k = -20.00 dB TOTAL = -20.40 dB (x0.0955) PCM5102A full scale is 2.1 Vrms, so at max volume Vout = 2.1 x 0.0955 = 0.201 Vrms at J1 Peak SPL = IEM dB/Vrms + 20*log10(Vout), and to convert a dB/mW spec: dB/Vrms = dB/mW + 10*log10(1000/Z) KZ Z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"
- note removed: "SHDN_SIGNAL LOW acts as setting the volume to a "true 0%" by shutting off the IEM amp. This is in contrast to the DAC Soft mute which acts as a mute toggle without changing the volume. Amp follows the pseudo-differential input configuration because the DAC output is a single-ended input."
