File: KiCad/RX_SKETCHES/dac.kicad_sch (KiCad schematic)
At the start: 14 parts, among them SW2 Interpolation Mode, SW3 DAC Soft Mute, U1 PCM5102

Commit message: Rewire RX hierarchical labels and mark proto DNP parts.
Keep the rotated WROOM-32U and breadboard I2S GPIOs, but attach
ESP_EN/IO0, UART, and BCK/DIN/LRCLK to the pins that actually sit
there after the 270° rotate. Move PCM5102 I2S off FMT/DEMP/XSMT,
put amp shutdown on ~{SHDN}, keep the datasheet 470R+2.2nF filter,
DNP the experimental pot pad and MAX97220A input resistors, and
switch schematic passives to 0805 for hand assembly.

Co-authored-by: luciano <dlmuschamp@users.noreply.github.com>
Parts:
- C13, C14, C15, C16, C17, C18, C19, C20, C21: footprint Capacitor_SMD:C_0201_0603Metric -> Capacitor_SMD:C_0805_2012Metric
- R16, R17: footprint Resistor_SMD:R_0201_0603Metric -> Resistor_SMD:R_0805_2012Metric
Connections:
- net BCK: now also U1.10 (DEMP); no longer U1.13 (BCK)
- net DIN: now also U1.17 (XSMT); no longer U1.14 (DIN)
- net GND: now also U1.13 (BCK), U1.15 (LRCK)
- net LRCLK: now also U1.16 (FMT); no longer U1.15 (LRCK)
- net at SW2.3 (A): now also SW3.1 (C)
- net at SW3.3 (A): now also U1.14 (DIN); no longer U1.17 (XSMT)
- no-connect marks 4 -> 1
Other:
- note added: "I2S on BCK / DIN / LRCK (not FMT / DEMP / XSMT). FMT and DEMP tied low = I2S, de-emphasis off. SCK grounded = PLL from BCK/LRCK. XSMT = SW3 soft mute. FLT = SW2 interpolation. OUTL/OUTR RC: 470R series + 2.2nF to GND (PCM5102 datasheet, assumed 10k load). MAX97220A Zin is ~10k, so this filter matches."
- moved on the sheet: SW3
Changed lines of the file:
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@@
 		(comment 3 "Soft Mute: XSMT LOW = Muted. XSMT HIGH = Unmuted. [Default]")
+	)
+	(text "I2S on BCK / DIN / LRCK (not FMT / DEMP / XSMT).\nFMT and DEMP tied low = I2S, de-emphasis off.\nSCK grounded = PLL from BCK/LRCK.\nXSMT = SW3 soft mute. FLT = SW2 interpolation.\n\nOUTL/OUTR RC: 470R series + 2.2nF to GND\n(PCM5102 datasheet, assumed 10k load).\nMAX97220A Zin is ~10k, so this filter matches."
+		(exclude_from_sim no)
+		(at 15.24 88.9 0)
+		(effects
+			(font
+				(size 1.27 1.27)
+			)
+			(justify left)
+		)
 	)
 	(text "DAC"
@@
 	)
 	(no_connect
-		(at 91.44 64.77)
-	)
-	(no_connect
-		(at 91.44 59.69)
-	)
-	(no_connect
-		(at 78.74 71.12)
-	)
-	(no_connect
 		(at 78.74 49.53)
 	)
@@
 	(wire
 		(pts
-			(xy 78.74 62.23) (xy 78.74 66.04)
+			(xy 78.74 44.45) (xy 78.74 46.99)
 		)
 		(stroke
@@
 	(wire
 		(pts
-			(xy 90.17 49.53) (xy 91.44 49.53)
+			(xy 90.17 59.69) (xy 91.44 59.69)
 		)
 		(stroke
@@
 	(wire
 		(pts
-			(xy 90.17 44.45) (xy 91.44 44.45)
+			(xy 90.17 64.77) (xy 91.44 64.77)
 		)
 		(stroke
@@
 	(wire
 		(pts
-			(xy 90.17 46.99) (xy 91.44 46.99)
+			(xy 90.17 62.23) (xy 91.44 62.23)
 		)
 		(stroke
@@
 	(wire
 		(pts
+			(xy 63.5 52.07) (xy 63.5 46.99)
+		)
+		(stroke
+			(width 0)
+			(type default)
+		)
+	)
+	(wire
+		(pts
 			(xy 104.14 26.67) (xy 104.14 24.13)
 		)
@@
 	(wire
 		(pts
-			(xy 63.5 68.58) (xy 68.58 68.58)
+			(xy 63.5 46.99) (xy 68.58 46.99)
 		)
 		(stroke
@@
 	(wire
 		(pts
-			(xy 78.74 62.23) (xy 91.44 62.23)
+			(xy 78.74 46.99) (xy 91.44 46.99)
 		)
 		(stroke
@@
 			(type default)
 		)
+	)
+	(wire
+		(pts
+			(xy 91.44 44.45) (xy 87.63 44.45)
+		)
+		(stroke
+			(width 0)
+			(type default)
+		)
+	)
+	(wire
+		(pts
+			(xy 87.63 44.45) (xy 87.63 49.53)
+		)
+		(stroke
+			(width 0)
+			(type default)
+		)
+	)
+	(wire
+		(pts
+			(xy 91.44 49.53) (xy 87.63 49.53)
+		)
+		(stroke
+			(width 0)
+			(type default)
+		)
+	)
+	(wire
+		(pts
+			(xy 87.63 49.53) (xy 87.63 52.07)
+		)
+		(stroke
+			(width 0)
+			(type default)
+		)
+	)
+	(junction
+		(at 87.63 49.53)
+		(diameter 0)
+		(color 0 0 0 0)
 	)
 	(hierarchical_label "DIN"
 		(shape input)
-		(at 90.17 46.99 180)
+		(at 90.17 62.23 180)
 		(effects
 			(font
@@
 	(hierarchical_label "LRCLK"
 		(shape input)
-		(at 90.17 44.45 180)
+		(at 90.17 64.77 180)
 		(effects
 			(font
@@
 	(hierarchical_label "BCK"
 		(shape input)
-		(at 90.17 49.53 180)
+		(at 90.17 59.69 180)
 		(effects
 			(font
@@
 			)
 		)
-		(property "Footprint" "Capacitor_SMD:C_0201_0603Metric"
+		(property "Footprint" "Capacitor_SMD:C_0805_2012Metric"
 			(at 166.0652 62.23 0)
 			(hide yes)
@@
 			)
 		)
-		(property "Footprint" "Resistor_SMD:R_0201_0603Metric"
+		(property "Footprint" "Resistor_SMD:R_0805_2012Metric"
 			(at 127.254 52.324 90)
 			(hide yes)
@@
 	(symbol
 		(lib_id "Switch:SW_Nidec_CAS-120A1")
-		(at 73.66 68.58 0)
+		(at 73.66 46.99 0)
 		(unit 1)
 		(body_style 1)
@@
 		(dnp no)
 		(property "Reference" "SW3"
-			(at 73.66 76.708 0)
+			(at 73.66 55.118 0)
 			(show_name no)
 			(do_not_autoplace no)
@@
 		)
 		(property "Value" "DAC Soft Mute"
-			(at 73.66 74.676 0)
+			(at 73.66 53.086 0)
 			(show_name no)
 			(do_not_autoplace no)
@@
 			)
 		)
-		(property "Footprint" "Capacitor_SMD:C_0201_0603Metric"
+		(property "Footprint" "Capacitor_SMD:C_0805_2012Metric"
 			(at 129.2352 76.2 0)
 			(hide yes)
@@
 			)
 		)
-		(property "Footprint" "Capacitor_SMD:C_0201_0603Metric"
+		(property "Footprint" "Capacitor_SMD:C_0805_2012Metric"
 			(at 120.3452 59.69 0)
 			(hide yes)
@@
 			)
 		)
-		(property "Footprint" "Capacitor_SMD:C_0201_0603Metric"
+		(property "Footprint" "Capacitor_SMD:C_0805_2012Metric"
 			(at 58.7248 49.53 0)
 			(hide yes)
@@
 			)
 		)
-		(property "Footprint" "Capacitor_SMD:C_0201_0603Metric"
+		(property "Footprint" "Capacitor_SMD:C_0805_2012Metric"
 			(at 119.0752 76.2 0)
 			(hide yes)
@@
 			)
 		)
-		(property "Footprint" "Capacitor_SMD:C_0201_0603Metric"
+		(property "Footprint" "Capacitor_SMD:C_0805_2012Metric"
 			(at 48.5648 49.53 0)
 			(hide yes)
@@
 			)
 		)
-		(property "Footprint" "Resistor_SMD:R_0201_0603Metric"
+		(property "Footprint" "Resistor_SMD:R_0805_2012Metric"
 			(at 127.254 37.084 90)
 			(hide yes)
@@
 			)
 		)
-		(property "Footprint" "Capacitor_SMD:C_0201_0603Metric"
+		(property "Footprint" "Capacitor_SMD:C_0805_2012Metric"
 			(at 139.3952 62.23 0)
 			(hide yes)
@@
 			)
 		)
-		(property "Footprint" "Capacitor_SMD:C_0201_0603Metric"
+		(property "Footprint" "Capacitor_SMD:C_0805_2012Metric"
 			(at 134.3152 48.26 0)
 			(hide yes)
@@
 			)
 		)
-		(property "Footprint" "Capacitor_SMD:C_0201_0603Metric"
+		(property "Footprint" "Capacitor_SMD:C_0805_2012Metric"
 			(at 154.6352 62.23 0)
 			(hide yes)

Commit message: Align RX passives and analog nets with the part datasheets.
Put every R/C on the 0805 HandSolder footprint. Rewire the PCM5102
470R filter onto OUTL/OUTR, decouple LDOO, and land the flying cap
on CAPP/CAPM. Move the headphone jack off PVSS/SVSS onto OUTL/OUTR
with a PVSS hold cap. Tie CP2102C VIO to VDD, pull RST up, add the
LM3940 0.47uF Cin, and pull IO0 up for normal boot.

Co-authored-by: luciano <dlmuschamp@users.noreply.github.com>
Parts:
- added C28: 0.1u, Capacitor_SMD:C_0805_2012Metric_Pad1.15x1.40mm_HandSolder, symbol Device:C
- C13, C14, C15, C16, C17, C18, C19, C20, C21: footprint Capacitor_SMD:C_0805_2012Metric -> Capacitor_SMD:C_0805_2012Metric_Pad1.15x1.40mm_HandSolder
- R16, R17: footprint Resistor_SMD:R_0805_2012Metric -> Resistor_SMD:R_0805_2012Metric_Pad1.20x1.40mm_HandSolder
Connections:
- net GND: now also C28.1
- net at R17.1, U1.7 (OUTR): now also C17.1, R16.1, U1.18 (LDOO), U1.6 (OUTL), C28.2
Other:
- note added: "I2S on BCK / DIN / LRCK (not FMT / DEMP / XSMT). FMT and DEMP tied low = I2S, de-emphasis off. SCK grounded = PLL from BCK/LRCK. XSMT = SW3 soft mute. FLT = SW2 interpolation. OUTL/OUTR (pins 6/7) -> 470R + 2.2nF to GND. LDOO (pin 18) has C28 0.1u to GND (datasheet). CAPP-CAPM flying cap hits pin ends. VNEG bulk stays. Do not attach the analog filter to LDOO."
- note removed: "I2S on BCK / DIN / LRCK (not FMT / DEMP / XSMT). FMT and DEMP tied low = I2S, de-emphasis off. SCK grounded = PLL from BCK/LRCK. XSMT = SW3 soft mute. FLT = SW2 interpolation. OUTL/OUTR RC: 470R series + 2.2nF to GND (PCM5102 datasheet, assumed 10k load). MAX97220A Zin is ~10k, so this filter matches."
