File: KiCad/RX_SKETCHES/dac.kicad_sch (KiCad schematic)
At the start: 15 parts, among them SW2 Interpolation Mode, SW3 DAC Soft Mute, U1 PCM5102

Commit message: WIP: RX schematic review — restore DAC/amp, fix ESP nets, log revisions.
Restore dac/amp from main after rotate damage, rename I2S net to DOUT,
mark amp gain Rs DNP, and record change/rationale in docs/hardware_revisions.org.

Co-authored-by: Cursor <cursoragent@cursor.com>
Parts:
- removed C28: 0.1u, Capacitor_SMD:C_0805_2012Metric_Pad1.15x1.40mm_HandSolder, symbol Device:C
- C13, C14, C15, C16, C17, C18, C19, C20, C21: footprint Capacitor_SMD:C_0805_2012Metric_Pad1.15x1.40mm_HandSolder -> Capacitor_SMD:C_0201_0603Metric
- R16, R17: footprint Resistor_SMD:R_0805_2012Metric_Pad1.20x1.40mm_HandSolder -> Resistor_SMD:R_0201_0603Metric
Connections:
- net DIN is gone; now on an unnamed net: U1.17 (XSMT)
- net BCK: now also U1.13 (BCK); no longer U1.10 (DEMP)
- net GND: no longer U1.13 (BCK), U1.15 (LRCK)
- net LRCLK: now also U1.15 (LRCK); no longer U1.16 (FMT)
- net at SW2.3 (A): no longer SW3.1 (C)
- net at SW3.3 (A): no longer U1.14 (DIN)
- new net: R17.1, U1.7 (OUTR)
- new net: C17.1, U1.18 (LDOO)
- new net: R16.1, U1.6 (OUTL)
- new net DOUT: U1.14 (DIN)
- no-connect marks 1 -> 4
Other:
- note removed: "I2S on BCK / DIN / LRCK (not FMT / DEMP / XSMT). FMT and DEMP tied low = I2S, de-emphasis off. SCK grounded = PLL from BCK/LRCK. XSMT = SW3 soft mute. FLT = SW2 interpolation. OUTL/OUTR (pins 6/7) -> 470R + 2.2nF to GND. LDOO (pin 18) has C28 0.1u to GND (datasheet). CAPP-CAPM flying cap hits pin ends. VNEG bulk stays. Do not attach the analog filter to LDOO."
- moved on the sheet: SW3

Commit message: RX: finish layout, retune gain/coupling, move ESD clamp to unswitched VBUS
Board now passes DRC with zero unconnected items and zero schematic-parity
issues. Remaining 16 violations are footprint-inherent (ESP32 module thermal
via array at 0.2 mm drill, USB-C NPTH-to-pad spacing) and are documented
rather than routed around.

Analog changes, with the reasoning captured in README.org and
docs/hardware_revisions.org so the numbers can be re-checked:

- Gain network populated at RF 4.7k / RIN 47k (-20 dB) instead of DNP 10k.
  Tames the DAC's 2.1 Vrms into sensitive IEMs, unloads the pot taper, and
  moves the coupling corner out of the audible band.
- Coupling caps C1-C4 0.47uF -> 1uF. Corner 7.2 Hz -> 3.4 Hz, and it halves
  the signal developed across the ceramic at 20 Hz, cutting Class-II
  dielectric distortion where it actually occurs.
- D1's third TVS channel moved off the switched +5V rail onto VBUS_RAW. The
  clamp has to sit on the connector pin that is exposed to a finger; behind
  the power switch it went open exactly when the board is most handled.
- SW3 soft mute: XSMT_SEL moved to the throw that puts mute on the south
  slide position. All three switches now follow one rule -- the open throw
  is the safe default (off / quality filter / muted).
- PCM5102 mode pins no longer float: FLT and XSMT get 100k pulldowns, DEMP
  and FMT strap to GND.
- C28 and the four mounting holes added to the schematic to clear parity
  errors against parts that only existed on the PCB.

Also adds a .gitignore so the 24 MB editor .history/ directory and ESP-IDF
build output stop showing up as untracked.

Co-authored-by: Cursor <cursoragent@cursor.com>
Parts:
- removed C18: 10u, Capacitor_SMD:C_0201_0603Metric, symbol Device:C
- added C12: 10u, Capacitor_SMD:C_0805_2012Metric_Pad1.18x1.45mm_HandSolder, symbol Device:C_Polarized
- added R31, R32: 100k, Resistor_SMD:R_0805_2012Metric_Pad1.20x1.40mm_HandSolder, symbol Device:R_US
- C13, C14, C15, C16, C17, C19, C20, C21: footprint Capacitor_SMD:C_0201_0603Metric -> Capacitor_SMD:C_0805_2012Metric_Pad1.18x1.45mm_HandSolder
- R16, R17: footprint Resistor_SMD:R_0201_0603Metric -> Resistor_SMD:R_0805_2012Metric_Pad1.20x1.40mm_HandSolder
- SW2: value Interpolation Mode -> FILTER_MODE; footprint Button_Switch_SMD:Nidec_Copal_CAS-120A -> Button_Switch_SMD:SW_SPDT_Shouhan_MSK12C02
- SW3: value DAC Soft Mute -> SOFT_MUTE; footprint Button_Switch_SMD:Nidec_Copal_CAS-120A -> Button_Switch_SMD:SW_SPDT_Shouhan_MSK12C02
Connections:
- net +3V3: now also C12.1
- net GND: now also U1.10 (DEMP), U1.16 (FMT), C12.2, R31.2, R32.2
- net FLT_SEL: now reaches SW2.1 (C), U1.11 (FLT)
- net FLT_SEL: now also R31.1
- net XSMT_SEL: now reaches SW3.1 (C)
- net XSMT_SEL: now also U1.17 (XSMT), R32.1
- net at SW3.3 (A): no longer U1.17 (XSMT)
- no-connect marks 4 -> 2
Other:
- note added: "AUDIO BANDWIDTH / FILTER AUDIT Only two reactive parts sit in the signal path. The rest of the chain is resistive, and the MAX97220 DirectDrive output is ground-referenced, so J1 needs no output cap and has none. 1) Reconstruction LP: R16/R17 470R + C20/C21 2.2nF, loaded by VR1 10k. R = 470||10k = 449R fc = 1/(2*pi*449*2.2n) = 161 kHz -> -0.07 dB @ 20 kHz 2) Input coupling HP: C1/C4 1uF into R_IN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"
- note added: "Must select interpolation mode before RX BOOT. Cannot change during operation."
- moved on the sheet: C13, C14, C15, C16, C17, C19, C20, C21, R16, R17, SW2, SW3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
