File: KiCad/RX_SKETCHES/dac.kicad_sch (KiCad schematic)
At the start: 14 parts, among them SW2 Interpolation Mode, SW3 DAC Soft Mute, U1 PCM5102

Commit message: RX v1: complete PCB layout, retune analog chain, fix ESD clamp placement
Brings the RX schematic and board up to a fabricable state. DRC is clean:
zero unconnected items, zero schematic-parity issues. The 16 remaining
violations are footprint-inherent and documented rather than worked around
(ESP32-WROOM thermal via array drilled 0.2 mm against a 0.3 mm rule, and
USB-C NPTH-to-pad spacing from the vendor land pattern).

Analog:
- Gain network populated at RF 4.7k / RIN 47k (-20 dB) rather than DNP 10k.
  Tames the PCM5102's 2.1 Vrms into sensitive IEMs, gives the 10k pot a
  4.7x loading ratio instead of 1:1, and lifts the coupling corner clear of
  the audible band.
- Coupling caps C1-C4 raised 0.47uF -> 1uF. Corner 7.2 Hz -> 3.4 Hz, and it
  halves the signal developed across the ceramic at 20 Hz, which is where
  Class-II dielectric distortion actually shows up.
- PCM5102 mode pins no longer float: 100k pulldowns on FLT and XSMT, with
  DEMP and FMT strapped to GND.

Power and protection:
- D1's third TVS channel moved off the switched +5V rail onto VBUS_RAW. An
  ESD clamp has to sit on the connector pin exposed to a finger; behind the
  power switch it disconnected exactly when the board is most likely to be
  handled. The off state is unaffected -- a TVS is open below its standoff
  voltage and SW4 still breaks the rail.
- All three slide switches now follow one rule: the open throw is the safe
  default (powered off / normal-latency filter / muted).

Housekeeping:
- C28 and mounting holes REF1-REF4 added to the schematic, clearing parity
  errors against parts that previously existed only on the PCB.
- Gain, loudness, and filter math written up in README.org with sources so
  the numbers can be re-derived; rationale logged in hardware_revisions.org.
- .gitignore now covers the editor .history/ directory and ESP-IDF build
  output, which were showing up as untracked noise.

Firmware and build artifacts are deliberately excluded from this commit.

Co-authored-b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
Parts:
- removed C18: 10u, Capacitor_SMD:C_0201_0603Metric, symbol Device:C
- added C12: 10u, Capacitor_SMD:C_0805_2012Metric_Pad1.18x1.45mm_HandSolder, symbol Device:C_Polarized
- added R31, R32: 100k, Resistor_SMD:R_0805_2012Metric_Pad1.20x1.40mm_HandSolder, symbol Device:R_US
- C13, C14, C15, C16, C17, C19, C20, C21: footprint Capacitor_SMD:C_0201_0603Metric -> Capacitor_SMD:C_0805_2012Metric_Pad1.18x1.45mm_HandSolder
- R16, R17: footprint Resistor_SMD:R_0201_0603Metric -> Resistor_SMD:R_0805_2012Metric_Pad1.20x1.40mm_HandSolder
- SW2: value Interpolation Mode -> FILTER_MODE; footprint Button_Switch_SMD:Nidec_Copal_CAS-120A -> Button_Switch_SMD:SW_SPDT_Shouhan_MSK12C02
- SW3: value DAC Soft Mute -> SOFT_MUTE; footprint Button_Switch_SMD:Nidec_Copal_CAS-120A -> Button_Switch_SMD:SW_SPDT_Shouhan_MSK12C02
Connections:
- net +3V3: now also C12.1
- net GND: now also U1.10 (DEMP), U1.16 (FMT), C12.2, R31.2, R32.2
- net FLT_SEL: now reaches SW2.1 (C), U1.11 (FLT)
- net FLT_SEL: now also R31.1
- net XSMT_SEL: now reaches SW3.1 (C)
- net XSMT_SEL: now also U1.17 (XSMT), R32.1
- net at SW3.3 (A): no longer U1.17 (XSMT)
- net DIN renamed DOUT
- no-connect marks 4 -> 2
Other:
- note added: "AUDIO BANDWIDTH / FILTER AUDIT Only two reactive parts sit in the signal path. The rest of the chain is resistive, and the MAX97220 DirectDrive output is ground-referenced, so J1 needs no output cap and has none. 1) Reconstruction LP: R16/R17 470R + C20/C21 2.2nF, loaded by VR1 10k. R = 470||10k = 449R fc = 1/(2*pi*449*2.2n) = 161 kHz -> -0.07 dB @ 20 kHz 2) Input coupling HP: C1/C4 1uF into R_IN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"
- note added: "Must select interpolation mode before RX BOOT. Cannot change during operation."
- moved on the sheet: C13, C14, C15, C16, C17, C19, C20, C21, R16, R17, SW2, SW3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
