File: KiCad/RX_SKETCHES/pwr_mgmt.kicad_sch (KiCad schematic)
At the start: 20 parts, among them J6 USB_C_Receptacle_USB2.0_16P, Q1 S8050, Q2 S8050, SW4 ON/OFF, U4 LM3940IMPX-3.3_NOPB, U5 CP2102C-Axx-xQFN24

Commit message: RX v1: complete PCB layout, retune analog chain, fix ESD clamp placement
Brings the RX schematic and board up to a fabricable state. DRC is clean:
zero unconnected items, zero schematic-parity issues. The 16 remaining
violations are footprint-inherent and documented rather than worked around
(ESP32-WROOM thermal via array drilled 0.2 mm against a 0.3 mm rule, and
USB-C NPTH-to-pad spacing from the vendor land pattern).

Analog:
- Gain network populated at RF 4.7k / RIN 47k (-20 dB) rather than DNP 10k.
  Tames the PCM5102's 2.1 Vrms into sensitive IEMs, gives the 10k pot a
  4.7x loading ratio instead of 1:1, and lifts the coupling corner clear of
  the audible band.
- Coupling caps C1-C4 raised 0.47uF -> 1uF. Corner 7.2 Hz -> 3.4 Hz, and it
  halves the signal developed across the ceramic at 20 Hz, which is where
  Class-II dielectric distortion actually shows up.
- PCM5102 mode pins no longer float: 100k pulldowns on FLT and XSMT, with
  DEMP and FMT strapped to GND.

Power and protection:
- D1's third TVS channel moved off the switched +5V rail onto VBUS_RAW. An
  ESD clamp has to sit on the connector pin exposed to a finger; behind the
  power switch it disconnected exactly when the board is most likely to be
  handled. The off state is unaffected -- a TVS is open below its standoff
  voltage and SW4 still breaks the rail.
- All three slide switches now follow one rule: the open throw is the safe
  default (powered off / normal-latency filter / muted).

Housekeeping:
- C28 and mounting holes REF1-REF4 added to the schematic, clearing parity
  errors against parts that previously existed only on the PCB.
- Gain, loudness, and filter math written up in README.org with sources so
  the numbers can be re-derived; rationale logged in hardware_revisions.org.
- .gitignore now covers the editor .history/ directory and ESP-IDF build
  output, which were showing up as untracked noise.

Firmware and build artifacts are deliberately excluded from this commit.

Co-authored-b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
Parts:
- added C30: 22u, Capacitor_SMD:C_0805_2012Metric_Pad1.18x1.45mm_HandSolder, symbol Device:C
- C22: value 22u -> 0.47u; footprint Capacitor_SMD:C_0201_0603Metric -> Capacitor_SMD:C_0805_2012Metric_Pad1.18x1.45mm_HandSolder
- C23, C24, C25, C26, C27: footprint Capacitor_SMD:C_0201_0603Metric -> Capacitor_SMD:C_0805_2012Metric_Pad1.18x1.45mm_HandSolder
- R11, R23, R24, R25, R26, R27, R7: footprint Resistor_SMD:R_0201_0603Metric -> Resistor_SMD:R_0805_2012Metric_Pad1.20x1.40mm_HandSolder
- SW4: footprint Button_Switch_SMD:Nidec_Copal_CAS-120A -> Button_Switch_SMD:SW_SPDT_Shouhan_MSK12C02
Connections:
- net +5V: now also C30.1; no longer D1.2 (K)
- net GND: now also C30.2
- net VBUS_RAW: now reaches J6.A4 (VBUS), J6.A9 (VBUS), J6.B4 (VBUS), J6.B9 (VBUS), SW4.2 (B)
- net VBUS_RAW: now also D1.2 (K)
Other:
- note added: "A01 G"
- note added: "CP2102C: VIO tied to VDD (+3V3). R29 1k pulls ~{RST} to VIO. R25/R26 are the VBUS divider (22.1k/47.5k)."
- note added: "LM3940: Cin >= 0.47uF (C30). Cout C23 = 33uF with ESR in the datasheet band. Prefer tantalum. A lone 0805 ceramic 33uF can be too-low ESR; add ~0.5 ohm series if C23 is ceramic."
- moved on the sheet: C22, C23, U4
