File: KiCad/RX_SKETCHES/pwr_mgmt.kicad_sch (KiCad schematic)
At the start: 22 parts, among them J6 USB_C_Receptacle_USB2.0_16P, Q1 S8050, Q2 S8050, SW4 ON/OFF, U4 LM3940IMPX-3.3_NOPB, U5 CP2102C-Axx-xQFN24

Commit message: WIP: RX schematic review — restore DAC/amp, fix ESP nets, log revisions.
Restore dac/amp from main after rotate damage, rename I2S net to DOUT,
mark amp gain Rs DNP, and record change/rationale in docs/hardware_revisions.org.

Co-authored-by: Cursor <cursoragent@cursor.com>
Parts:
- removed C31: 0.47u, Capacitor_SMD:C_0805_2012Metric_Pad1.15x1.40mm_HandSolder, symbol Device:C
- removed R29: 1k, Resistor_SMD:R_0805_2012Metric_Pad1.20x1.40mm_HandSolder, symbol Device:R_US
- added C30: 22u, Capacitor_SMD:C_0805_2012Metric_Pad1.15x1.40mm_HandSolder, symbol Device:C
- C22: value 22u -> 0.47u
Connections:
- net +5V: now also C30.1
- net GND: now also C30.2
Other:
- note added: "A01 G"
- note added: "CP2102C: VIO tied to VDD (+3V3). R29 1k pulls ~{RST} to VIO. R25/R26 are the VBUS divider (22.1k/47.5k)."
- note added: "LM3940: Cin >= 0.47uF (C30). Cout C23 = 33uF with ESR in the datasheet band. Prefer tantalum. A lone 0805 ceramic 33uF can be too-low ESR; add ~0.5 ohm series if C23 is ceramic."
- note removed: "CP2102C: VIO tied to VDD (+3V3).\nR29 1k pulls ~{RST} to VIO.\nR25/R26 are the VBUS divider (22.1k/47.5k)."
- note removed: "LM3940: Cin >= 0.47uF (C31). Cout C23 = 33uF\nwith ESR in the datasheet band. Prefer tantalum.\nA lone 0805 ceramic 33uF can be too-low ESR;\nadd ~0.5 ohm series if C23 is ceramic."
- moved on the sheet: C22, C23, U4

Commit message: RX: finish layout, retune gain/coupling, move ESD clamp to unswitched VBUS
Board now passes DRC with zero unconnected items and zero schematic-parity
issues. Remaining 16 violations are footprint-inherent (ESP32 module thermal
via array at 0.2 mm drill, USB-C NPTH-to-pad spacing) and are documented
rather than routed around.

Analog changes, with the reasoning captured in README.org and
docs/hardware_revisions.org so the numbers can be re-checked:

- Gain network populated at RF 4.7k / RIN 47k (-20 dB) instead of DNP 10k.
  Tames the DAC's 2.1 Vrms into sensitive IEMs, unloads the pot taper, and
  moves the coupling corner out of the audible band.
- Coupling caps C1-C4 0.47uF -> 1uF. Corner 7.2 Hz -> 3.4 Hz, and it halves
  the signal developed across the ceramic at 20 Hz, cutting Class-II
  dielectric distortion where it actually occurs.
- D1's third TVS channel moved off the switched +5V rail onto VBUS_RAW. The
  clamp has to sit on the connector pin that is exposed to a finger; behind
  the power switch it went open exactly when the board is most handled.
- SW3 soft mute: XSMT_SEL moved to the throw that puts mute on the south
  slide position. All three switches now follow one rule -- the open throw
  is the safe default (off / quality filter / muted).
- PCM5102 mode pins no longer float: FLT and XSMT get 100k pulldowns, DEMP
  and FMT strap to GND.
- C28 and the four mounting holes added to the schematic to clear parity
  errors against parts that only existed on the PCB.

Also adds a .gitignore so the 24 MB editor .history/ directory and ESP-IDF
build output stop showing up as untracked.

Co-authored-by: Cursor <cursoragent@cursor.com>
Parts:
- C22, C23, C24, C25, C26, C27, C30: footprint Capacitor_SMD:C_0805_2012Metric_Pad1.15x1.40mm_HandSolder -> Capacitor_SMD:C_0805_2012Metric_Pad1.18x1.45mm_HandSolder
- SW4: footprint Button_Switch_SMD:Nidec_Copal_CAS-120A -> Button_Switch_SMD:SW_SPDT_Shouhan_MSK12C02
Connections:
- net +5V: no longer D1.2 (K)
- net VBUS_RAW: now reaches J6.A4 (VBUS), J6.A9 (VBUS), J6.B4 (VBUS), J6.B9 (VBUS), SW4.2 (B)
- net VBUS_RAW: now also D1.2 (K)
Changed lines of the file:
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@@
 	)
 	(junction
+		(at 55.88 25.4)
+		(diameter 0)
+		(color 0 0 0 0)
+	)
+	(junction
 		(at 86.36 49.53)
 		(diameter 0)
@@
 	)
 	(junction
-		(at 81.28 22.86)
-		(diameter 0)
-		(color 0 0 0 0)
-	)
-	(junction
 		(at 30.48 128.27)
 		(diameter 0)
@@
 	(wire
 		(pts
-			(xy 125.73 86.36) (xy 128.27 86.36)
+			(xy 55.88 17.78) (xy 55.88 25.4)
 		)
 		(stroke
@@
 	(wire
 		(pts
-			(xy 77.47 22.86) (xy 81.28 22.86)
+			(xy 77.47 22.86) (xy 86.36 22.86)
 		)
 		(stroke
@@
 	(wire
 		(pts
-			(xy 140.97 34.29) (xy 146.05 34.29)
+			(xy 55.88 25.4) (xy 59.69 25.4)
 		)
 		(stroke
@@
 	(wire
 		(pts
-			(xy 86.36 22.86) (xy 86.36 41.91)
+			(xy 140.97 34.29) (xy 146.05 34.29)
 		)
 		(stroke
@@
 	(wire
 		(pts
-			(xy 138.43 55.88) (xy 147.32 55.88)
+			(xy 86.36 22.86) (xy 86.36 41.91)
 		)
 		(stroke
@@
 	(wire
 		(pts
-			(xy 81.28 22.86) (xy 81.28 74.93)
+			(xy 138.43 55.88) (xy 147.32 55.88)
 		)
 		(stroke
@@
 	(wire
 		(pts
-			(xy 81.28 22.86) (xy 86.36 22.86)
+			(xy 24.13 128.27) (xy 30.48 128.27)
 		)
 		(stroke
@@
 	(wire
 		(pts
-			(xy 24.13 128.27) (xy 30.48 128.27)
+			(xy 50.8 58.42) (xy 53.34 58.42)
 		)
 		(stroke
@@
 	(wire
 		(pts
-			(xy 50.8 58.42) (xy 53.34 58.42)
+			(xy 53.34 71.12) (xy 53.34 68.58)
 		)
 		(stroke
@@
 	(wire
 		(pts
-			(xy 53.34 71.12) (xy 53.34 68.58)
+			(xy 81.28 73.66) (xy 81.28 74.93)
 		)
 		(stroke
@@
 	(wire
 		(pts
-			(xy 113.03 81.28) (xy 113.03 82.55)
-		)
-		(stroke
-			(width 0)
-			(type default)
-		)
-	)
-	(wire
-		(pts
 			(xy 157.48 71.12) (xy 160.02 71.12)
 		)
@@
 	(wire
 		(pts
-			(xy 50.8 25.4) (xy 59.69 25.4)
+			(xy 50.8 25.4) (xy 55.88 25.4)
 		)
 		(stroke
@@
 	(wire
 		(pts
+			(xy 80.01 73.66) (xy 81.28 73.66)
+		)
+		(stroke
+			(width 0)
+			(type default)
+		)
+	)
+	(wire
+		(pts
 			(xy 50.8 71.12) (xy 53.34 71.12)
 		)
@@
 		)
 	)
+	(label "VBUS_RAW"
+		(at 80.01 73.66 180)
+		(effects
+			(font
+				(size 1.27 1.27)
+			)
+			(justify right bottom)
+		)
+	)
+	(label "VBUS_RAW"
+		(at 55.88 17.78 0)
+		(effects
+			(font
+				(size 1.27 1.27)
+			)
+			(justify left bottom)
+		)
+	)
 	(hierarchical_label "TXD"
 		(shape output)
@@
 			)
 		)
-		(property "Footprint" "Capacitor_SMD:C_0805_2012Metric_Pad1.15x1.40mm_HandSolder"
+		(property "Footprint" "Capacitor_SMD:C_0805_2012Metric_Pad1.18x1.45mm_HandSolder"
 			(at 105.1052 33.02 0)
 			(hide yes)
@@
 			)
 		)
-		(property "Footprint" "Capacitor_SMD:C_0805_2012Metric_Pad1.15x1.40mm_HandSolder"
+		(property "Footprint" "Capacitor_SMD:C_0805_2012Metric_Pad1.18x1.45mm_HandSolder"
 			(at 25.0952 123.19 0)
 			(hide yes)
@@
 			)
 		)
-		(property "Footprint" "Capacitor_SMD:C_0805_2012Metric_Pad1.15x1.40mm_HandSolder"
+		(property "Footprint" "Capacitor_SMD:C_0805_2012Metric_Pad1.18x1.45mm_HandSolder"
 			(at 115.2652 33.02 0)
 			(hide yes)
@@
 			)
 		)
-		(property "Footprint" "Button_Switch_SMD:Nidec_Copal_CAS-120A"
+		(property "Footprint" "Button_Switch_SMD:SW_SPDT_Shouhan_MSK12C02"
 			(at 64.77 35.56 0)
 			(hide yes)
@@
 			)
 		)
-		(property "Footprint" "Capacitor_SMD:C_0805_2012Metric_Pad1.15x1.40mm_HandSolder"
+		(property "Footprint" "Capacitor_SMD:C_0805_2012Metric_Pad1.18x1.45mm_HandSolder"
 			(at 136.8552 33.02 0)
 			(hide yes)
@@
 			)
 		)
-		(property "Footprint" "Capacitor_SMD:C_0805_2012Metric_Pad1.15x1.40mm_HandSolder"
+		(property "Footprint" "Capacitor_SMD:C_0805_2012Metric_Pad1.18x1.45mm_HandSolder"
 			(at 75.8952 123.19 0)
 			(hide yes)
@@
 			)
 		)
-		(property "Footprint" "Capacitor_SMD:C_0805_2012Metric_Pad1.15x1.40mm_HandSolder"
+		(property "Footprint" "Capacitor_SMD:C_0805_2012Metric_Pad1.18x1.45mm_HandSolder"
 			(at 31.4452 123.19 0)
 			(hide yes)
@@
 			)
 		)
-		(property "Footprint" "Capacitor_SMD:C_0805_2012Metric_Pad1.15x1.40mm_HandSolder"
+		(property "Footprint" "Capacitor_SMD:C_0805_2012Metric_Pad1.18x1.45mm_HandSolder"
 			(at 147.0152 33.02 0)
 			(hide yes)

Commit message: RX v1: map JLCPCB parts, fix LM3940 bulk cap, add production export
Retune the LM3940 input divider to 22k/47k and swap C23 to an EIA-3528
tantalum so the regulator meets its minimum ESR and stays stable.

Every SMT part now carries an LCSC number in the plugin's project.db, with
the ESP32 module and the mechanical/reference parts excluded from assembly
so the order stays on Economic pricing. Includes the generated Gerbers,
BOM, and CPL, plus the clean DRC/ERC reports.

Co-authored-by: Cursor <cursoragent@cursor.com>
Parts:
- C23: footprint Capacitor_SMD:C_0805_2012Metric_Pad1.18x1.45mm_HandSolder -> Capacitor_Tantalum_SMD:CP_EIA-3528-12_Kemet-T_HandSolder
- R25: value 22.1k -> 22k
- R26: value 47.5k -> 47k
Changed lines of the file:
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@@
 			)
 		)
-		(property "Value" "47.5k"
+		(property "Value" "47k"
 			(at 88.9 55.8799 0)
 			(show_name no)
@@
 			)
 		)
-		(property "Value" "22.1k"
+		(property "Value" "22k"
 			(at 88.9 46.9899 0)
 			(show_name no)
@@
 			)
 		)
-		(property "Footprint" "Capacitor_SMD:C_0805_2012Metric_Pad1.18x1.45mm_HandSolder"
+		(property "Footprint" "Capacitor_Tantalum_SMD:CP_EIA-3528-12_Kemet-T_HandSolder"
 			(at 75.8952 123.19 0)
-			(hide yes)
-			(show_name no)
-			(do_not_autoplace no)
+			(show_name no)
+			(do_not_autoplace no)
