File: KiCad/RX_SKETCHES/vol_ctrl.kicad_sch (KiCad schematic)
At the start: 6 parts

Commit message: Rewire RX hierarchical labels and mark proto DNP parts.
Keep the rotated WROOM-32U and breadboard I2S GPIOs, but attach
ESP_EN/IO0, UART, and BCK/DIN/LRCLK to the pins that actually sit
there after the 270° rotate. Move PCM5102 I2S off FMT/DEMP/XSMT,
put amp shutdown on ~{SHDN}, keep the datasheet 470R+2.2nF filter,
DNP the experimental pot pad and MAX97220A input resistors, and
switch schematic passives to 0805 for hand assembly.

Co-authored-by: luciano <dlmuschamp@users.noreply.github.com>
Parts:
- R18, R19, R20, R21: footprint Resistor_SMD:R_0201_0603Metric -> Resistor_SMD:R_0805_2012Metric; now not fitted
- R22: footprint Resistor_SMD:R_0201_0603Metric -> Resistor_SMD:R_0805_2012Metric
Connections:
- net PRE_POT_IN_L is gone; now on net DAC_OUT_L: R18.2, R19.1, VR1.3 (CW1)
- net PRE_POT_IN_R is gone; now on net DAC_OUT_R: R20.2, R21.1, VR1.6 (CW2)
Other:
- note added: "PCM5102 datasheet filter lives on the DAC sheet: DAC_OUT -- 470R -- PRE_POT, 2.2nF from that node to GND. That network assumes ~10 kOhm. MAX97220A Zin is ~10 kOhm. R18/R20 1k and R19/R21 10R are the old experimental 40 dB pad. They are DNP. Wires short the 1k positions so the pot sees the filtered DAC_OUT directly. Leave the 10R pads empty (do not shunt PRE_POT to GND)."
Changed lines of the file:
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@@
 		(company "damian m")
 		(comment 1 "Data: TX -> RX -> DAC -> AMP-> 3.5mm Jack.")
-		(comment 2 "AMP_IN_L/R follows a voltage divdier to lower volume to safer levels before hitting AMP.")
+		(comment 2 "DAC_OUT uses the PCM5102 470R + 2.2nF filter (on the DAC sheet), then the dual-gang pot. Experimental 1k/10R pad is DNP.")
 		(comment 3 "Volume Knob with integrated off switch to kill amp from playing any audio. ")
 		(comment 4 "POST_POT_IN_R/L becomes the input to the amp.")
@@
 			(width 0)
 			(type default)
+		)
+	)
+	(wire
+		(pts
+			(xy 97.79 25.4) (xy 97.79 38.1)
+		)
+		(stroke
+			(width 0)
+			(type default)
+		)
+	)
+	(wire
+		(pts
+			(xy 110.49 25.4) (xy 110.49 38.1)
+		)
+		(stroke
+			(width 0)
+			(type default)
+		)
+	)
+	(text "PCM5102 datasheet filter lives on the DAC sheet:\nDAC_OUT -- 470R -- PRE_POT, 2.2nF from that node to GND.\nThat network assumes ~10 kOhm. MAX97220A Zin is ~10 kOhm.\n\nR18/R20 1k and R19/R21 10R are the old experimental\n40 dB pad. They are DNP. Wires short the 1k positions\nso the pot sees the filtered DAC_OUT directly.\nLeave the 10R pads empty (do not shunt PRE_POT to GND)."
+		(exclude_from_sim no)
+		(at 20.32 20.32 0)
+		(effects
+			(font
+				(size 1.27 1.27)
+			)
+			(justify left)
 		)
 	)
@@
 		(on_board yes)
 		(in_pos_files yes)
-		(dnp no)
+		(dnp yes)
 		(fields_autoplaced yes)
 		(property "Reference" "R18"
@@
 			)
 		)
-		(property "Footprint" "Resistor_SMD:R_0201_0603Metric"
+		(property "Footprint" "Resistor_SMD:R_0805_2012Metric"
 			(at 98.806 30.734 90)
 			(hide yes)
@@
 			)
 		)
-		(property "Footprint" "Resistor_SMD:R_0201_0603Metric"
+		(property "Footprint" "Resistor_SMD:R_0805_2012Metric"
 			(at 122.936 87.884 90)
 			(hide yes)
@@
 		(on_board yes)
 		(in_pos_files yes)
-		(dnp no)
+		(dnp yes)
 		(fields_autoplaced yes)
 		(property "Reference" "R21"
@@
 			)
 		)
-		(property "Footprint" "Resistor_SMD:R_0201_0603Metric"
+		(property "Footprint" "Resistor_SMD:R_0805_2012Metric"
 			(at 111.506 45.974 90)
 			(hide yes)
@@
 		(on_board yes)
 		(in_pos_files yes)
-		(dnp no)
+		(dnp yes)
 		(fields_autoplaced yes)
 		(property "Reference" "R19"
@@
 			)
 		)
-		(property "Footprint" "Resistor_SMD:R_0201_0603Metric"
+		(property "Footprint" "Resistor_SMD:R_0805_2012Metric"
 			(at 98.806 45.974 90)
 			(hide yes)
@@
 		(on_board yes)
 		(in_pos_files yes)
-		(dnp no)
+		(dnp yes)
 		(fields_autoplaced yes)
 		(property "Reference" "R20"
@@
 			)
 		)
-		(property "Footprint" "Resistor_SMD:R_0201_0603Metric"
+		(property "Footprint" "Resistor_SMD:R_0805_2012Metric"
 			(at 111.506 30.734 90)
 			(hide yes)

Commit message: Align RX passives and analog nets with the part datasheets.
Put every R/C on the 0805 HandSolder footprint. Rewire the PCM5102
470R filter onto OUTL/OUTR, decouple LDOO, and land the flying cap
on CAPP/CAPM. Move the headphone jack off PVSS/SVSS onto OUTL/OUTR
with a PVSS hold cap. Tie CP2102C VIO to VDD, pull RST up, add the
LM3940 0.47uF Cin, and pull IO0 up for normal boot.

Co-authored-by: luciano <dlmuschamp@users.noreply.github.com>
Parts:
- R18, R19, R20, R21, R22: footprint Resistor_SMD:R_0805_2012Metric -> Resistor_SMD:R_0805_2012Metric_Pad1.20x1.40mm_HandSolder
Changed lines of the file:
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@@
 			)
 		)
-		(property "Footprint" "Resistor_SMD:R_0805_2012Metric"
+		(property "Footprint" "Resistor_SMD:R_0805_2012Metric_Pad1.20x1.40mm_HandSolder"
 			(at 98.806 30.734 90)
 			(hide yes)
@@
 			)
 		)
-		(property "Footprint" "Resistor_SMD:R_0805_2012Metric"
+		(property "Footprint" "Resistor_SMD:R_0805_2012Metric_Pad1.20x1.40mm_HandSolder"
 			(at 122.936 87.884 90)
 			(hide yes)
@@
 			)
 		)
-		(property "Footprint" "Resistor_SMD:R_0805_2012Metric"
+		(property "Footprint" "Resistor_SMD:R_0805_2012Metric_Pad1.20x1.40mm_HandSolder"
 			(at 111.506 45.974 90)
 			(hide yes)
@@
 			)
 		)
-		(property "Footprint" "Resistor_SMD:R_0805_2012Metric"
+		(property "Footprint" "Resistor_SMD:R_0805_2012Metric_Pad1.20x1.40mm_HandSolder"
 			(at 98.806 45.974 90)
 			(hide yes)
@@
 			)
 		)
-		(property "Footprint" "Resistor_SMD:R_0805_2012Metric"
+		(property "Footprint" "Resistor_SMD:R_0805_2012Metric_Pad1.20x1.40mm_HandSolder"
 			(at 111.506 30.734 90)
 			(hide yes)
