File: KiCad/TX_SKETCHES/ESP_32_IEM_RIG_TX_VER_1.0.kicad_pcb (KiCad board)
At the start: 2 copper layers, 0 parts

Commit message: Ship RX+TX v1 boards: routed PCBs, JLCPCB exports, README for order spin.
Freeze electrical intent for fab (Gerbers/BOM/CPL), document firmware design philosophy and summer timeline, and drop stale ERC/DRC/fab clutter.

Co-authored-by: Cursor <cursoragent@cursor.com>
Parts:
- added C11: 0.1u, Capacitor_SMD:C_0805_2012Metric_Pad1.18x1.45mm_HandSolder, F.Cu at (91.0, 53.4)
- added C12: 10uF, Capacitor_SMD:C_0805_2012Metric_Pad1.18x1.45mm_HandSolder, F.Cu at (117.5, 79.8)
- added C13: 1uF, Capacitor_SMD:C_0805_2012Metric_Pad1.18x1.45mm_HandSolder, F.Cu at (130.3, 89.2)
- added C14: 1nF, Capacitor_SMD:C_0805_2012Metric_Pad1.18x1.45mm_HandSolder, F.Cu at (126.4, 91.8)
- added C15: 1uF, Capacitor_SMD:C_0805_2012Metric_Pad1.18x1.45mm_HandSolder, F.Cu at (130.3, 80.9)
- added C16: 1nF, Capacitor_SMD:C_0805_2012Metric_Pad1.18x1.45mm_HandSolder, F.Cu at (126.6, 78.3)
- added C17: 0.1u, Capacitor_SMD:C_0805_2012Metric_Pad1.18x1.45mm_HandSolder, F.Cu at (119.5, 79.8)
- added C18: 10uF, Capacitor_SMD:C_0805_2012Metric_Pad1.18x1.45mm_HandSolder, F.Cu at (113.5, 82.7)
- added C19: 0.1u, Capacitor_SMD:C_0805_2012Metric_Pad1.18x1.45mm_HandSolder, F.Cu at (115.5, 82.7)
- added C20: 10uF, Capacitor_SMD:C_0805_2012Metric_Pad1.18x1.45mm_HandSolder, F.Cu at (113.5, 86.5)
- added C21: 0.1u, Capacitor_SMD:C_0805_2012Metric_Pad1.18x1.45mm_HandSolder, F.Cu at (115.5, 86.5)
- added C22: 0.47u, Capacitor_SMD:C_0805_2012Metric_Pad1.18x1.45mm_HandSolder, F.Cu at (62.8, 66.8)
- added C23: 33u, Capacitor_Tantalum_SMD:CP_EIA-3528-12_Kemet-T_HandSolder, F.Cu at (68.3, 67.6)
- added C24: 4.7u, Capacitor_SMD:C_0805_2012Metric_Pad1.18x1.45mm_HandSolder, F.Cu at (77.0, 83.5)
- added C25: 0.1u, Capacitor_SMD:C_0805_2012Metric_Pad1.18x1.45mm_HandSolder, F.Cu at (77.0, 81.5)
- added C26: 4.7u, Capacitor_SMD:C_0805_2012Metric_Pad1.18x1.45mm_HandSolder, F.Cu at (79.8, 77.3)
- added C27: 0.1u, Capacitor_SMD:C_0805_2012Metric_Pad1.18x1.45mm_HandSolder, F.Cu at (79.8, 79.3)
- added C30: 22u, Capacitor_SMD:C_0805_2012Metric_Pad1.18x1.45mm_HandSolder, F.Cu at (64.8, 66.8)
- added C31: 0.1u, Capacitor_SMD:C_0805_2012Metric_Pad1.18x1.45mm_HandSolder, F.Cu at (91.3, 76.0)
- added C5: 22u, Capacitor_SMD:C_0805_2012Metric_Pad1.18x1.45mm_HandSolder, F.Cu at (89.0, 53.5)
- added D1: SP0503BAHT, Package_TO_SOT_SMD:SOT-143, F.Cu at (81.8, 49.6)
- added J2: AudioJack3, Connector_Audio:Jack_3.5mm_CUI_SJ-3523-SMT_Horizontal, F.Cu at (141.3, 84.8)
- added J6: USB_C_Receptacle_USB2.0_16P, Connector_USB:USB_C_Receptacle_GCT_USB4105-xx-A_16P_TopMnt_Horizontal, F.Cu at (81.8, 43.0)
- added Q1: S8050, Package_TO_SOT_SMD:SOT-23, F.Cu at (89.3, 79.5)
- added Q2: S8050, Package_TO_SOT_SMD:SOT-23, F.Cu at (89.3, 85.1)
- added R11: 10k, Resistor_SMD:R_0805_2012Metric_Pad1.20x1.40mm_HandSolder, F.Cu at (86.3, 85.2)
- added R12: 120, Resistor_SMD:R_0805_2012Metric_Pad1.20x1.40mm_HandSolder, F.Cu at (126.5, 89.2)
- added R13: 120, Resistor_SMD:R_0805_2012Metric_Pad1.20x1.40mm_HandSolder, F.Cu at (126.5, 80.9)
- added R14: 100k, Resistor_SMD:R_0805_2012Metric_Pad1.20x1.40mm_HandSolder, F.Cu at (126.5, 82.9)
- added R15: 100k, Resistor_SMD:R_0805_2012Metric_Pad1.20x1.40mm_HandSolder, F.Cu at (126.5, 87.0)
- added R16: 100k, Resistor_SMD:R_0805_2012Metric_Pad1.20x1.40mm_HandSolder, F.Cu at (126.5, 85.0)
- added R23: 5.1k, Resistor_SMD:R_0805_2012Metric_Pad1.20x1.40mm_HandSolder, F.Cu at (88.3, 46.0)
- added R24: 5.1k, Resistor_SMD:R_0805_2012Metric_Pad1.20x1.40mm_HandSolder, F.Cu at (75.3, 46.0)
- added R25: 22k, Resistor_SMD:R_0805_2012Metric_Pad1.20x1.40mm_HandSolder, F.Cu at (75.0, 87.7)
- added R26: 47k, Resistor_SMD:R_0805_2012Metric_Pad1.20x1.40mm_HandSolder, F.Cu at (77.5, 87.7)
- added R27: 1k, Resistor_SMD:R_0805_2012Metric_Pad1.20x1.40mm_HandSolder, F.Cu at (79.5, 87.7)
- added R30: 10k, Resistor_SMD:R_0805_2012Metric_Pad1.20x1.40mm_HandSolder, F.Cu at (92.3, 79.2)
- added R7: 10k, Resistor_SMD:R_0805_2012Metric_Pad1.20x1.40mm_HandSolder, F.Cu at (86.3, 79.5)
- added R8: 10k, Resistor_SMD:R_0805_2012Metric_Pad1.20x1.40mm_HandSolder, F.Cu at (73.5, 76.0)
- added REF1: MountingHole_2.7mm_M2.5, MountingHole:MountingHole_2.7mm_M2.5, F.Cu at (96.5, 86.4)
- added REF2: MountingHole_2.7mm_M2.5, MountingHole:MountingHole_2.7mm_M2.5, F.Cu at (96.3, 49.4)
- added REF3: MountingHole_2.7mm_M2.5, MountingHole:MountingHole_2.7mm_M2.5, F.Cu at (70.5, 49.4)
- added REF4: MountingHole_2.7mm_M2.5, MountingHole:MountingHole_2.7mm_M2.5, F.Cu at (63.9, 90.4)
- added SW4: ON/OFF, Button_Switch_SMD:SW_SPDT_Shouhan_MSK12C02, F.Cu at (62.3, 43.4)
- added U1: PCM1808PWG4, PCM1808PWG4:SOP65P640X120-14N, F.Cu at (120.5, 84.5)
- added U2: ESP32-WROOM-32U, RF_Module:ESP32-WROOM-32U, F.Cu at (84.1, 65.2)
- added U4: LM3940IMPX-3.3_NOPB, LM3940IMPX-3.3_NOPB:SOT230P700X180-4N, F.Cu at (64.8, 60.6)
- added U5: CP2102C-Axx-xQFN24, Package_DFN_QFN:WQFN-24-1EP_4x4mm_P0.5mm_EP2.45x2.45mm, F.Cu at (82.3, 83.0)
Routing:
- net +5V: track 0.00 -> 140.0 mm, vias 0 -> 2
- net +3V3: track 0.00 -> 130.0 mm, vias 0 -> 2
- net /ADC/SCK: track 0.00 -> 85.0 mm, vias 0 -> 4
- net GND: track 0.00 -> 71.9 mm, vias 0 -> 36
- net /ADC/BCK: track 0.00 -> 55.7 mm, vias 0 -> 2
- net /ADC/DIN: track 0.00 -> 54.5 mm, vias 0 -> 2
- net /ADC/LRCK: track 0.00 -> 52.6 mm, vias 0 -> 4
- net Net-(U5-D-): track 0.00 -> 38.9 mm, vias 0 -> 3
- net Net-(U5-D+): track 0.00 -> 38.5 mm, vias 0 -> 2
- net /Power Management/VBUS_RAW: track 0.00 -> 33.7 mm, vias 0 -> 2
- net /ESP Transmitter/ESP_EN: track 0.00 -> 29.0 mm, vias 0 -> 2
- net Net-(U5-VDD): track 0.00 -> 20.9 mm, vias 0 -> 2
- net /ADC/V_IN_R: track 0.00 -> 17.6 mm
- net /ESP Transmitter/RXD: track 0.00 -> 13.1 mm, vias 0 -> 2
- net /ADC/RIGHT: track 0.00 -> 11.8 mm
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- added copper zone on B.Cu, net GND
- added copper zone on F.Cu, net GND
Other:
- board outline added: 90.5 x 55.2 mm
- board text added: "Designed by Damian Muschamp | https://github.com/dlmuschamp/ESP32IEMPack.git Transmitter Unit"

Commit message: Refresh TX/RX silk artwork and regenerate JLCPCB gerbers.
Cosmetic pass: silkscreen, QR codes, font, and screw hole moves — BOM/CPL unchanged.

Co-authored-by: Cursor <cursoragent@cursor.com>
Parts:
- moved REF2 0.81 mm to (95.5, 49.5)
Other:
- board text added: "3V3"
- board text added: "5V"
- board text added: "5V IN"
- board text added: "ADC"
- board text added: "ANALOG INPUT"
- board text added: "DESIGNER : [ DAMIAN LUCIANO MUSCHAMP ]r GITHUB : [ https://github.com/dlmuschamp/ESP32IEMPack.git ]r SYSTEM : [ ESP32 WIRELESS TRANSMITTER IEM PACK ]r PROTOCOL : [ ESP-NOW (UNENCRYPTED) ]r PAYLOAD : [ 720 SAMPLES (1440 B) UNCOMPRESSED ]r RATE : [ 48 kHz ]r FORMAT : [ STEREO ]r REV_DATE : [ 2026-09-02 ]"
- board text added: "ESD"
- board text added: "ESP32U WROOM"
- board text added: "LDO"
- board text added: "ON/OFF"
- board text added: "USB-C TO UART"
- board text removed: "Designed by Damian Muschamp | https://github.com/dlmuschamp/ESP32IEMPack.git Transmitter Unit"
